File: V1.1/V1.1.kicad_pcb (KiCad board)
At the start: 2 copper layers, 76.2 x 80.2 mm, 43 parts, among them SW1 SW_Push, U1 ATmega32U4-AU, U2 SRV05-4, Y1 16MHz

Commit message: Fixed routing even further
Routing:
- net Net-(R3-Pad2): track 23.1 -> 24.9 mm
- net +5V: track 101.9 -> 103.4 mm
