File: V1.1/KiCad/V1.1.sch (KiCad schematic (older format))
At the start: 43 parts, among them SW1 SW_Push, U1 ATmega32U4-AU, U2 SRV05-4, Y1 16MHz

Commit message: Added images, organized files
Parts:
- MX1, MX10, MX11, MX12, MX2, MX3, MX4, MX5, MX6, MX7, MX8, MX9: symbol MX_Alps_Hybrid:MX-NoLED -> V1.1-rescue:MX-NoLED-MX_Alps_Hybrid
- USB1: symbol Type-C:HRO-TYPE-C-31-M-12 -> V1.1-rescue:HRO-TYPE-C-31-M-12-Type-C
Changed lines of the file:
@@
 D-
 $Comp
-L Type-C:HRO-TYPE-C-31-M-12 USB1
+L V1.1-rescue:HRO-TYPE-C-31-M-12-Type-C USB1
 U 1 1 6185DB88
 P 4300 1500
@@
 $EndComp
 $Comp
-L MX_Alps_Hybrid:MX-NoLED MX1
+L V1.1-rescue:MX-NoLED-MX_Alps_Hybrid MX1
 U 1 1 6187DC71
 P 5450 3450
@@
 $EndComp
 $Comp
-L MX_Alps_Hybrid:MX-NoLED MX2
+L V1.1-rescue:MX-NoLED-MX_Alps_Hybrid MX2
 U 1 1 61888BA2
 P 6000 3450
@@
 $EndComp
 $Comp
-L MX_Alps_Hybrid:MX-NoLED MX3
+L V1.1-rescue:MX-NoLED-MX_Alps_Hybrid MX3
 U 1 1 6188BBFE
 P 6500 3450
@@
 $EndComp
 $Comp
-L MX_Alps_Hybrid:MX-NoLED MX4
+L V1.1-rescue:MX-NoLED-MX_Alps_Hybrid MX4
 U 1 1 6188BC0B
 P 7050 3450
@@
 $EndComp
 $Comp
-L MX_Alps_Hybrid:MX-NoLED MX5
+L V1.1-rescue:MX-NoLED-MX_Alps_Hybrid MX5
 U 1 1 618A611C
 P 5450 4150
@@
 $EndComp
 $Comp
-L MX_Alps_Hybrid:MX-NoLED MX6
+L V1.1-rescue:MX-NoLED-MX_Alps_Hybrid MX6
 U 1 1 618A6129
 P 6000 4150
@@
 $EndComp
 $Comp
-L MX_Alps_Hybrid:MX-NoLED MX7
+L V1.1-rescue:MX-NoLED-MX_Alps_Hybrid MX7
 U 1 1 618A6136
 P 6500 4150
@@
 $EndComp
 $Comp
-L MX_Alps_Hybrid:MX-NoLED MX8
+L V1.1-rescue:MX-NoLED-MX_Alps_Hybrid MX8
 U 1 1 618A6143
 P 7050 4150
@@
 $EndComp
 $Comp
-L MX_Alps_Hybrid:MX-NoLED MX9
+L V1.1-rescue:MX-NoLED-MX_Alps_Hybrid MX9
 U 1 1 618ADC8C
 P 5450 4800
@@
 $EndComp
 $Comp
-L MX_Alps_Hybrid:MX-NoLED MX10
+L V1.1-rescue:MX-NoLED-MX_Alps_Hybrid MX10
 U 1 1 618ADC99
 P 6000 4800
@@
 $EndComp
 $Comp
-L MX_Alps_Hybrid:MX-NoLED MX11
+L V1.1-rescue:MX-NoLED-MX_Alps_Hybrid MX11
 U 1 1 618ADCA6
 P 6500 4800
@@
 $EndComp
 $Comp
-L MX_Alps_Hybrid:MX-NoLED MX12
+L V1.1-rescue:MX-NoLED-MX_Alps_Hybrid MX12
 U 1 1 618ADCB3
 P 7050 4800
@@
 Text GLabel 3450 3950 2    50   Input ~ 0
 COL3
-Text GLabel 3450 3250 2    50   Input ~ 0
+Text GLabel 3450 3050 2    50   Input ~ 0
 ROW0
 Text GLabel 3450 3150 2    50   Input ~ 0
 ROW1
-Text GLabel 3450 3050 2    50   Input ~ 0
+Text GLabel 3450 3250 2    50   Input ~ 0
 ROW2
 $EndSCHEMATC
